File: PCB/RenewableRegulator_MPPT_PCB_2017/powersupply.sch (KiCad schematic (older format))
At the start: 15 parts, among them P11 TP_GND, P12 TP_5V, P13 TP_10V, U2 LMR16006, U3 MCP1702-50

Commit message: First version MPPT PCB
Parts:
- C8: footprint matts_components:C1_wide_lg_pad -> REInnovationFootprint:cond_1
- P11, P12, P13: footprint matts_components:1pin_0_8mm -> REInnovationFootprint:tp
- U3: footprint matts_components:TO92_MCP9701_matt -> REInnovationFootprint:TH_TO92-EBC_large_pad_u3
Changed lines of the file:
@@
 LIBS:power
 LIBS:device
+LIBS:conn
 LIBS:matts_components
-LIBS:conn
 LIBS:RenewableRegulator_MPPT_PCB_2017-cache
 EELAYER 25 0
@@
 $Descr A4 11693 8268
 encoding utf-8
-Sheet 3 5
+Sheet 2 5
 Title "Renewable Regulator"
 Date "2017-04-04"
@@
 F 0 "C8" H 5075 2900 50  0000 L CNN
 F 1 "100nf" H 5075 2700 50  0000 L CNN
-F 2 "matts_components:C1_wide_lg_pad" H 5088 2650 50  0001 C CNN
+F 2 "REInnovationFootprint:cond_1" H 5088 2650 50  0001 C CNN
 F 3 "" H 5050 2800 50  0000 C CNN
 	1    5050 2800
@@
 F 0 "U3" H 5050 5054 60  0000 C CNN
 F 1 "MCP1702-50" H 4900 5450 60  0000 C CNN
-F 2 "matts_components:TO92_MCP9701_matt" H 4900 5250 60  0001 C CNN
+F 2 "REInnovationFootprint:TH_TO92-EBC_large_pad_u3" H 4900 5250 60  0001 C CNN
 F 3 "http://docs-europe.electrocomponents.com/webdocs/0a77/0900766b80a77df4.pdf" H 4900 5250 60  0001 C CNN
 F 4 "~" H 4900 5250 60  0000 C CNN "Notes"
@@
 F 0 "P13" H 6750 3050 50  0000 C CNN
 F 1 "TP_10V" V 6850 2950 50  0000 C CNN
-F 2 "matts_components:1pin_0_8mm" H 6750 2950 50  0001 C CNN
+F 2 "REInnovationFootprint:tp" H 6750 2950 50  0001 C CNN
 F 3 "" H 6750 2950 50  0000 C CNN
 	1    6750 2950
@@
 F 0 "P12" H 6300 5150 50  0000 C CNN
 F 1 "TP_5V" V 6400 5050 50  0000 C CNN
-F 2 "matts_components:1pin_0_8mm" H 6300 5050 50  0001 C CNN
+F 2 "REInnovationFootprint:tp" H 6300 5050 50  0001 C CNN
 F 3 "" H 6300 5050 50  0000 C CNN
 	1    6300 5050
@@
 F 0 "P11" H 5950 6050 50  0000 C CNN
 F 1 "TP_GND" V 6050 5950 50  0000 C CNN
-F 2 "matts_components:1pin_0_8mm" H 5950 5950 50  0001 C CNN
+F 2 "REInnovationFootprint:tp" H 5950 5950 50  0001 C CNN
 F 3 "" H 5950 5950 50  0000 C CNN
 	1    5950 5950
