File: PCB/RenewableRegulatorPCB_2017/RenewableRegulatorPCB_2017.kicad_pcb (KiCad board)
At the start: 2 copper layers, 101.3 x 90.8 mm, 62 parts, among them J1 TEMP, J2 Arduino_Nano, P1 INPUT, P10 TP_FET, P11 TP_GND, P12 TP_5V, P13 TP_10V, P2 Vref?, P3 MicroSD, P4 A6_7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

Commit message: Last version of regulator PCB
Other:
- net class Default: trace_width 2 -> 0.5
Changed lines of the file:
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@@
     (thickness 1.6002)
     (drawings 24)
-    (tracks 574)
+    (tracks 576)
     (zones 0)
     (modules 62)
@@
   )
   (setup
-    (last_trace_width 2)
+    (last_trace_width 0.5)
     (trace_clearance 0.127)
     (zone_clearance 0.508)
@@
     (mod_text_size 1.524 1.524)
     (mod_text_width 0.3048)
-    (pad_size 3 3)
-    (pad_drill 3)
+    (pad_size 1.2 1.2)
+    (pad_drill 0.7)
     (pad_to_mask_clearance 0.254)
     (aux_axis_origin 88.9 90.805)
@@
   (net_class Default "This is the default net class."
     (clearance 0.127)
-    (trace_width 2)
+    (trace_width 0.5)
     (via_dia 0.889)
     (via_drill 0.635)
@@
     )
   )
+  (module REInnovationFootprint:TH_Inductor2 (layer Front)
+    (at 95.885 64.135)
+    (descr "Condensateur polarise")
+    (tags CP)
+    (fp_text reference L1 (at 0 -4.064 180) (layer F.SilkS)
+      (effects (font (size 1.016 1.016) (thickness 0.2032)))
+    )
+    (fp_text value 22uH (at 0 1.524) (layer F.SilkS) hide
+      (effects (font (size 1.016 1.016) (thickness 0.2032)))
+    )
+    (fp_circle (center 0 0) (end 0 -3) (layer F.SilkS) (width 0.15))
+    (pad 1 thru_hole circle (at -2.5 0) (size 2.032 2.032) (drill 0.8001) (layers *.Cu *.Mask F.SilkS)
+      (net 14 "Net-(C8-Pad2)"))
+    (pad 2 thru_hole circle (at 2.5 0) (size 2.032 2.032) (drill 0.8001) (layers *.Cu *.Mask F.SilkS)
+      (net 10 "/Power Supply/+10V"))
+    (model discret/c_vert_c2v10.wrl
+      (at (xyz 0 0 0))
+      (scale (xyz 1 1 1))
+      (rotate (xyz 0 0 0))
+    )
+  )
   (module REInnovationFootprint:TO92_MCP9701_matt2 (layer Front)
     (at 100.965 72.39)
@@
     (fp_arc (start 2.7025 -2.954) (end 2.7025 -0.254) (angle 90) (layer F.SilkS) (width 0.15))
     (fp_arc (start 2.7025 -2.954) (end 5.4025 -2.954) (angle 90) (layer F.SilkS) (width 0.15))
-    (pad GND thru_hole rect (at 4.064 -2.413) (size 1.2 1.2) (drill 0.7) (layers *.Cu *.Mask F.SilkS)
+    (pad GND thru_hole rect (at 4.064 -2.413) (size 1 1) (drill 0.6) (layers *.Cu *.Mask F.SilkS)
       (net 2 GND))
-    (pad VO thru_hole circle (at 1.524 -2.413) (size 1.2 1.2) (drill 0.7) (layers *.Cu *.Mask F.SilkS)
+    (pad VO thru_hole circle (at 1.524 -2.413) (size 1 1) (drill 0.6) (layers *.Cu *.Mask F.SilkS)
       (net 1 +5V))
-    (pad VI thru_hole circle (at 2.794 -2.413) (size 1.2 1.2) (drill 0.7) (layers *.Cu *.Mask F.SilkS)
+    (pad VI thru_hole circle (at 2.794 -2.413) (size 1 1) (drill 0.6) (layers *.Cu *.Mask F.SilkS)
       (net 10 "/Power Supply/+10V"))
     (model discret/to98.wrl
@@
     )
   )
-  (module REInnovationFootprint:TH_Inductor2 (layer Front)
-    (at 95.885 64.135)
-    (descr "Condensateur polarise")
-    (tags CP)
-    (fp_text reference L1 (at 0 -4.064 180) (layer F.SilkS)
-      (effects (font (size 1.016 1.016) (thickness 0.2032)))
-    )
-    (fp_text value 22uH (at 0 1.524) (layer F.SilkS) hide
-      (effects (font (size 1.016 1.016) (thickness 0.2032)))
-    )
-    (fp_circle (center 0 0) (end 0 -3) (layer F.SilkS) (width 0.15))
-    (pad 1 thru_hole circle (at -2.5 0) (size 2.032 2.032) (drill 0.8001) (layers *.Cu *.Mask F.SilkS)
-      (net 14 "Net-(C8-Pad2)"))
-    (pad 2 thru_hole circle (at 2.5 0) (size 2.032 2.032) (drill 0.8001) (layers *.Cu *.Mask F.SilkS)
-      (net 10 "/Power Supply/+10V"))
-    (model discret/c_vert_c2v10.wrl
-      (at (xyz 0 0 0))
-      (scale (xyz 1 1 1))
-      (rotate (xyz 0 0 0))
-    )
-  )
   (gr_text re-innovation.co.uk (at 161.925 78.486 90) (layer Back)
     (effects (font (size 2.032 1.524) (thickness 0.3048)) (justify mirror))
@@
   (segment (start 99.06 52.07) (end 99.06 53.911) (width 0.5) (layer Front) (net 1))
   (segment (start 99.06 53.911) (end 98.79 54.181) (width 0.5) (layer Front) (net 1))
+  (segment (start 104.14 72.39) (end 104.14 71.882) (width 0.5) (layer Front) (net 2))
+  (segment (start 105.029 70.993) (end 105.029 69.977) (width 0.5) (layer Front) (net 2) (status 800000))
+  (segment (start 104.14 71.882) (end 105.029 70.993) (width 0.5) (layer Front) (net 2))
   (segment (start 84.455 73.025) (end 83.185 73.025) (width 0.5) (layer Front) (net 2))
   (segment (start 82.55 72.39) (end 81.28 72.39) (width 0.5) (layer Front) (net 2))
@@
   (segment (start 101.6 52.07) (end 101.6 53.371) (width 0.5) (layer Front) (net 2))
   (segment (start 101.6 53.371) (end 100.79 54.181) (width 0.5) (layer Front) (net 2))
-  (segment (start 105.537 69.723) (end 105.0925 70.1675) (width 0.5) (layer Front) (net 2))
   (segment (start 104.14 85.09) (end 103.545 85.685) (width 0.5) (layer Front) (net 2))
   (segment (start 103.545 85.685) (end 102.235 85.685) (width 0.5) (layer Front) (net 2))
@@
   (segment (start 68.58 72.39) (end 70.485 70.485) (width 0.5) (layer Front) (net 2))
   (segment (start 70.485 70.485) (end 73.065 70.485) (width 0.5) (layer Front) (net 2))
-  (segment (start 105.0925 70.1675) (end 105.0925 70.8025) (width 0.5) (layer Front) (net 2))
-  (segment (start 105.0925 70.8025) (end 104.14 71.755) (width 0.5) (layer Front) (net 2))
-  (segment (start 104.14 71.755) (end 104.14 82.55) (width 0.5) (layer Front) (net 2))
+  (segment (start 104.14 72.39) (end 104.14 82.55) (width 0.5) (layer Front) (net 2))
   (segment (start 104.14 82.55) (end 104.14 85.09) (width 0.5) (layer Front) (net 2))
   (segment (start 104.14 85.09) (end 104.14 85.217) (width 0.5) (layer Front) (net 2))
@@
   (segment (start 79.502 103.378) (end 86.36 103.378) (width 2) (layer Front) (net 6))
   (segment (start 77.47 105.41) (end 79.502 103.378) (width 2) (layer Front) (net 6))
-  (segment (start 106.045 95.25) (end 114.3 95.25) (width 2) (layer Front) (net 7) (status 400000))
-  (segment (start 114.3 97.155) (end 114.3 95.25) (width 2) (layer Front) (net 7) (status 400000))
+  (segment (start 106.045 95.25) (end 114.3 95.25) (width 2) (layer Front) (net 7))
+  (segment (start 114.3 97.155) (end 114.3 95.25) (width 2) (layer Front) (net 7))
   (segment (start 114.3 95.25) (end 114.3 94.615) (width 2) (layer Front) (net 7))
   (segment (start 114.3 94.615) (end 114.9096 94.0054) (width 2) (layer Front) (net 7))
-  (segment (start 114.9096 94.0054) (end 116.586 94.0054) (width 2) (layer Front) (net 7) (status 800000))
+  (segment (start 114.9096 94.0054) (end 116.586 94.0054) (width 2) (layer Front) (net 7))
   (segment (start 99.1 102.235) (end 99.1 96.861) (width 1) (layer Back) (net 7))
   (segment (start 100.711 95.25) (end 106.045 95.25) (width 1) (layer Back) (net 7))
@@
   (segment (start 78.74 53.975) (end 78.74 57.785) (width 0.5) (layer Back) (net 16))
   (segment (start 76.2 51.435) (end 78.74 53.975) (width 0.5) (layer Back) (net 16))
-  (segment (start 104.14 91.44) (end 116.5606 91.44) (width 2) (layer Front) (net 17) (status C00000))
-  (segment (start 116.5606 91.44) (end 116.586 91.4654) (width 2) (layer Front) (net 17) (status C00000))
+  (segment (start 104.14 91.44) (end 116.5606 91.44) (width 2) (layer Front) (net 17))
+  (segment (start 116.5606 91.44) (end 116.586 91.4654) (width 2) (layer Front) (net 17))
   (segment (start 130.81 59.69) (end 130.81 60.198) (width 0.5) (layer Front) (net 18))
   (segment (start 148.59 67.818) (end 148.59 66.04) (width 0.5) (layer Front) (net 18))
@@
   (segment (start 93.98 53.371) (end 94.79 54.181) (width 0.5) (layer Front) (net 34))
   (segment (start 94.79 54.181) (end 94.821 54.181) (width 0.5) (layer Front) (net 34))
-  (segment (start 96.79 54.181) (end 96.79 55.61) (width 0.5) (layer Front) (net 35))
+  (segment (start 95.0595 74.168) (end 95.0595 57.9755) (width 0.5) (layer Back) (net 35))
+  (segment (start 96.79 56.118) (end 96.79 54.181) (width 0.5) (layer Front) (net 35))
+  (segment (start 94.996 57.912) (end 96.79 56.118) (width 0.5) (layer Front) (net 35))
+  (via (at 94.996 57.912) (size 0.889) (drill 0.635) (layers Front Back) (net 35))
+  (segment (start 95.0595 57.9755) (end 94.996 57.912) (width 0.5) (layer Back) (net 35))
+  (segment (start 95.0595 74.1045) (end 95.0595 74.168) (width 0.5) (layer Back) (net 35))
   (segment (start 105.41 76.835) (end 109.22 76.835) (width 0.5) (layer Front) (net 35))
   (via (at 105.41 76.835) (size 0.889) (drill 0.635) (layers Front Back) (net 35))
@@
   (segment (start 99.06 76.2) (end 99.695 76.835) (width 0.5) (layer Back) (net 35))
   (segment (start 97.155 76.2) (end 99.06 76.2) (width 0.5) (layer Back) (net 35))
-  (segment (start 94.615 73.66) (end 97.155 76.2) (width 0.5) (layer Back) (net 35))
-  (segment (start 94.615 57.785) (end 94.615 73.66) (width 0.5) (layer Back) (net 35))
-  (via (at 94.615 57.785) (size 0.889) (drill 0.635) (layers Front Back) (net 35))
-  (segment (start 96.79 55.61) (end 94.615 57.785) (width 0.5) (layer Front) (net 35))
+  (segment (start 95.0595 74.1045) (end 97.155 76.2) (width 0.5) (layer Back) (net 35))
   (segment (start 96.52 52.07) (end 96.52 53.911) (width 0.5) (layer Front) (net 35))
   (segment (start 96.52 53.911) (end 96.79 54.181) (width 0.5) (layer Front) (net 35))
